File: attic/planbook-keyboard/planbook-keyboard.kicad_pcb (KiCad board)
At the start: 2 copper layers, 154 x 84.5 mm, 143 parts, among them J1 USB, J2 UART, J3 AUX, SW1 Choc, SW10 Choc, SW11 Choc, SW12 Choc, SW13 Choc, SW14 Choc, SW15 Choc, SW16 Choc, SW17 Choc, SW18 Choc, SW19 Choc, SW2 Choc, SW20 Choc, SW21 Choc, SW22 Choc, SW23 Choc, SW24 Choc, SW25 Choc, SW26 Choc, SW27 Choc, SW28 Choc, SW29 Choc, SW3 Choc, SW30 Choc, SW31 Choc, SW32 Choc, SW33 Choc, SW34 Choc, SW35 Choc, SW36 Choc, SW37 Choc, SW38 Choc, SW39 Choc, SW4 Choc, SW40 Choc, SW41 Choc, SW42 Choc, SW43 Choc, SW44 Choc, SW45 Choc, SW46 Choc, SW47 Choc, SW48 Choc, SW49 Choc, SW5 Choc, SW50 Choc, SW51 Choc, SW52 Choc, SW53 Choc, SW54 Choc, SW55 Choc, SW56 RESET, SW6 Choc, SW7 Choc, SW8 Choc, SW9 Choc, U1 MCP1700-3302E_SOT23, U2 ATMEGA32U4-AU, Y1 16MHz

Commit message: Fix remaining MNT and branding references
- Fixed remaining MNT references in KiCad files and firmware
- Updated function names and constants to use PlanBook naming
- Fixed include headers and function declarations
- Updated remaining branding references in documentation

Generated with [Devin](https://devin.ai)

Co-Authored-By: Devin <158243242+devin-ai-integration[bot]@users.noreply.github.com>
Parts:
- GFX1, GFX2: value MNT -> PlanBook
Changed lines of the file:
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@@
   (page A4)
   (title_block
-    (title "MNT PlanBook Keyboard")
+    (title "PlanBook Keyboard")
     (date 2021-05-12)
     (rev D-1)
-    (company "MNT Research GmbH")
+    (company "PlanBook Project")
     (comment 1 "Lukas F. Hartmann")
     (comment 2 "CERN OHL-S 2.0")
@@
       (effects (font (size 1.524 1.524) (thickness 0.3)) (justify mirror))
     )
-    (fp_text value MNT (at 0.75 0) (layer B.SilkS) hide
+    (fp_text value PlanBook (at 0.75 0) (layer B.SilkS) hide
       (effects (font (size 1.524 1.524) (thickness 0.3)) (justify mirror))
     )
@@
       (effects (font (size 1.524 1.524) (thickness 0.3)) (justify mirror))
     )
-    (fp_text value MNT (at 0.75 0) (layer B.SilkS) hide
+    (fp_text value PlanBook (at 0.75 0) (layer B.SilkS) hide
       (effects (font (size 1.524 1.524) (thickness 0.3)) (justify mirror))
     )

Commit message: Replace PCB logos with PlanBook text
- Removed all badge footprint graphics from PCB files
- Added "PlanBook" text in same positions with default font
- Updated footprint library files to use simple text instead of complex logos
- Updated schematic footprint references to empty strings
- Text uses font size 1.5x1.5 with thickness 0.3
- Maintained exact positions and rotations from original footprints

Generated with [Devin](https://devin.ai)

Co-Authored-By: Devin <158243242+devin-ai-integration[bot]@users.noreply.github.com>
Parts:
- removed GFX2: PlanBook, footprints:mpre-badge-d1
Other:
- board text added: "PlanBook"
