File: planbook-keyboard-kailh-ortho/planbook-kbd-mcu.sch (KiCad schematic (older format))
At the start: 28 parts, among them J1 USB, J2 UART, J3 AUX, SW61 RESET, U1 ATMEGA32U4-AU, U1 MCP1700-3302E_SOT23, Y1 16MHz

Commit message: Fix remaining MNT and branding references
- Fixed remaining MNT references in KiCad files and firmware
- Updated function names and constants to use PlanBook naming
- Fixed include headers and function declarations
- Updated remaining branding references in documentation

Generated with [Devin](https://devin.ai)

Co-Authored-By: Devin <158243242+devin-ai-integration[bot]@users.noreply.github.com>
Parts:
- GFX1, GFX2: value MNT -> PlanBook
Changed lines of the file:
@@
 P 4750 7150
 F 0 "GFX1" H 4850 7196 50  0000 L CNN
-F 1 "MNT" H 4850 7105 50  0000 L CNN
+F 1 "PlanBook" H 4850 7105 50  0000 L CNN
 F 2 "footprints:planbook" H 4750 7150 50  0001 C CNN
 F 3 "~" H 4750 7150 50  0001 C CNN
@@
 P 5150 7150
 F 0 "GFX2" H 5250 7196 50  0000 L CNN
-F 1 "MNT" H 5250 7105 50  0000 L CNN
+F 1 "PlanBook" H 5250 7105 50  0000 L CNN
 F 2 "footprints:mpre-badge-d1" H 5150 7150 50  0001 C CNN
 F 3 "~" H 5150 7150 50  0001 C CNN
