File: planbook-keyboard-kailh-ortho/planbook-kbd-mcu.kicad_sch (KiCad schematic)
At the start: 51 parts, among them J1 Conn_01x06_Female, J2 USB, J3 UART, J4 AUX, J61 UART, SW65 SW_HWB, SW66 SW_RST, U12 AP22815A, U2 RP2040, U3 W25Q32JVSS, Y1 12MHz 12pF

Commit message: Fix remaining MNT and branding references
- Fixed remaining MNT references in KiCad files and firmware
- Updated function names and constants to use PlanBook naming
- Fixed include headers and function declarations
- Updated remaining branding references in documentation

Generated with [Devin](https://devin.ai)

Co-Authored-By: Devin <158243242+devin-ai-integration[bot]@users.noreply.github.com>
Parts:
- GFX1, GFX2: value MNT -> PlanBook
Changed lines of the file:
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@@
 			)
 		)
-		(property "Value" "MNT"
+		(property "Value" "PlanBook"
 			(at 113.03 231.013 0)
 			(effects
@@
 			)
 		)
-		(property "Value" "MNT"
+		(property "Value" "PlanBook"
 			(at 113.03 237.363 0)
 			(effects

Commit message: Replace PCB logos with PlanBook text
- Removed all badge footprint graphics from PCB files
- Added "PlanBook" text in same positions with default font
- Updated footprint library files to use simple text instead of complex logos
- Updated schematic footprint references to empty strings
- Text uses font size 1.5x1.5 with thickness 0.3
- Maintained exact positions and rotations from original footprints

Generated with [Devin](https://devin.ai)

Co-Authored-By: Devin <158243242+devin-ai-integration[bot]@users.noreply.github.com>
Parts:
- GFX2: footprint footprints:pref-keyboard15-badge -> (none)
Changed lines of the file:
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@@
 			)
 		)
-		(property "Footprint" "footprints:pref-keyboard15-badge"
+		(property "Footprint" ""
 			(at 110.49 236.22 0)
 			(effects
