File: planbook-keyboard-kailh-ortho/planbook-keyboard-kailh-ortho.kicad_pcb (KiCad board)
At the start: 4 copper layers, 194.4 x 114.3 mm, 309 parts, among them J1 Conn_01x06_Female, J2 USB, J3 UART, J4 AUX, J61 UART, SW1 Choc, SW10 Choc, SW11 Choc, SW12 Choc, SW13 Choc, SW14 Choc, SW15 Choc, SW16 Choc, SW17 Choc, SW18 Choc, SW19 Choc, SW2 Choc, SW20 Choc, SW21 Choc, SW22 Choc, SW23 Choc, SW24 Choc, SW25 Choc, SW26 Choc, SW27 Choc, SW28 Choc, SW29 Choc, SW3 Choc, SW30 Choc, SW31 Choc, SW32 Choc, SW33 Choc, SW34 Choc, SW35 Choc, SW36 Choc, SW37 Choc, SW38 Choc, SW39 Choc, SW4 Choc, SW40 Choc, SW41 Choc, SW42 Choc, SW43 Choc, SW44 Choc, SW45 Choc, SW46 Choc, SW47 Choc, SW48 Choc, SW49 Choc, SW5 Choc, SW50 Choc, SW51 Choc, SW52 Choc, SW53 Choc, SW54 Choc, SW55 Choc, SW56 Choc, SW57 Choc, SW58 Choc, SW59 Choc, SW6 Choc, SW60 Choc, SW61 Choc, SW62 Choc, SW63 Choc, SW64 Choc, SW65 SW_HWB, SW66 SW_RST, SW7 Choc, SW8 Choc, SW9 Choc, U1 SN74LV1T34DCK, U12 AP22815A, U2 RP2040, U3 W25Q32JVSS, Y1 12MHz 12pF

Commit message: Fix remaining MNT and branding references
- Fixed remaining MNT references in KiCad files and firmware
- Updated function names and constants to use PlanBook naming
- Fixed include headers and function declarations
- Updated remaining branding references in documentation

Generated with [Devin](https://devin.ai)

Co-Authored-By: Devin <158243242+devin-ai-integration[bot]@users.noreply.github.com>
Parts:
- GFX1, GFX2: value MNT -> PlanBook
Changed lines of the file:
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@@
 			)
 		)
-		(property "Value" "MNT"
+		(property "Value" "PlanBook"
 			(at 0.75 0 0)
 			(layer "B.SilkS")
@@
 			)
 		)
-		(property "Value" "MNT"
+		(property "Value" "PlanBook"
 			(at 0.75 0 0)
 			(layer "B.SilkS")

Commit message: Replace PCB logos with PlanBook text
- Removed all badge footprint graphics from PCB files
- Added "PlanBook" text in same positions with default font
- Updated footprint library files to use simple text instead of complex logos
- Updated schematic footprint references to empty strings
- Text uses font size 1.5x1.5 with thickness 0.3
- Maintained exact positions and rotations from original footprints

Generated with [Devin](https://devin.ai)

Co-Authored-By: Devin <158243242+devin-ai-integration[bot]@users.noreply.github.com>
Parts:
- removed GFX2: PlanBook, footprints:pref-keyboard15-badge
Other:
- board text added: "PlanBook"
