File: planbook-keyboard-kailh-ortho/planbook-keyboard-kailh-ortho.kicad_pcb (KiCad board)
At the start: 4 copper layers, 194.4 x 114.3 mm, 308 parts, among them J1 Conn_01x06_Female, J2 USB, J3 UART, J4 AUX, J61 UART, SW1 Choc, SW10 Choc, SW11 Choc, SW12 Choc, SW13 Choc, SW14 Choc, SW15 Choc, SW16 Choc, SW17 Choc, SW18 Choc, SW19 Choc, SW2 Choc, SW20 Choc, SW21 Choc, SW22 Choc, SW23 Choc, SW24 Choc, SW25 Choc, SW26 Choc, SW27 Choc, SW28 Choc, SW29 Choc, SW3 Choc, SW30 Choc, SW31 Choc, SW32 Choc, SW33 Choc, SW34 Choc, SW35 Choc, SW36 Choc, SW37 Choc, SW38 Choc, SW39 Choc, SW4 Choc, SW40 Choc, SW41 Choc, SW42 Choc, SW43 Choc, SW44 Choc, SW45 Choc, SW46 Choc, SW47 Choc, SW48 Choc, SW49 Choc, SW5 Choc, SW50 Choc, SW51 Choc, SW52 Choc, SW53 Choc, SW54 Choc, SW55 Choc, SW56 Choc, SW57 Choc, SW58 Choc, SW59 Choc, SW6 Choc, SW60 Choc, SW61 Choc, SW62 Choc, SW63 Choc, SW64 Choc, SW65 SW_HWB, SW66 SW_RST, SW7 Choc, SW8 Choc, SW9 Choc, U1 SN74LV1T34DCK, U12 AP22815A, U2 RP2040, U3 W25Q32JVSS, Y1 12MHz 12pF

Commit message: Phase 1: PCB design rules standardization
- Created standardized design rules document (planbook-design-rules.kicad_dru)
- Added comprehensive design rules documentation (DESIGN_RULES.md)
- Standardized board thickness to 1.6mm across all PCBs for mechanical strength
- Standardized copper finish to ENIG for better reliability
- Standardized pad-to-mask clearance to 0.05mm for manufacturing
- Updated layer stackup specifications for consistency

This provides a foundation for consistent manufacturing and performance improvements.

Note: Tooling holes and fiducials require KiCad GUI placement to avoid interfering with existing components.

Generated with [Devin](https://devin.ai)

Co-Authored-By: Devin <158243242+devin-ai-integration[bot]@users.noreply.github.com>
Other:
- rule pad_to_mask_clearance: 0 -> 0.05
Changed lines of the file:
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@@
 				(type "Bottom Silk Screen")
 			)
-			(copper_finish "None")
+			(copper_finish "ENIG")
 			(dielectric_constraints no)
 		)
-		(pad_to_mask_clearance 0)
+		(pad_to_mask_clearance 0.05)
 		(allow_soldermask_bridges_in_footprints no)
 		(tenting front back)

Commit message: Phase 2 & 3: PCB performance improvements and implementation guides
Implemented:
- Added ground stitching vias around board edges (214 vias total across 4 PCBs)
  - planbook-motherboard: 48 vias (10mm spacing)
  - planbook-charger: 26 vias (8mm spacing)
  - planbook-keyboard-kailh-ortho: 76 vias (8mm spacing)
  - planbook-wifi: 64 vias (5mm spacing)
- Via specifications: 0.3mm drill, 0.6mm diameter, connected to GND
- Improves EMI performance and grounding

Created comprehensive implementation guides:
- PHASE2_DECOUPLING_GUIDE.md: RP2040 decoupling capacitor recommendations
- PHASE2_ESD_PROTECTION_GUIDE.md: ESD protection for USB, SD card, keyboard, etc.
- PHASE3_THERMAL_MANAGEMENT_GUIDE.md: Thermal via recommendations for hot components
- PHASE3_COPPER_POUR_GUIDE.md: Copper pour improvements for heat dissipation
- PHASE3_LED_OPTIMIZATION_GUIDE.md: LED current limiting resistor optimization
- GROUND_STITCHING_VIAS_SUMMARY.md: Summary of ground stitching via additions

Guides require KiCad GUI implementation for component additions and modifications.

Generated with [Devin](https://devin.ai)

Co-Authored-By: Devin <158243242+devin-ai-integration[bot]@users.noreply.github.com>
Routing:
- net GND: vias 258 -> 334
