File: planbook-charger/planbook-charger.kicad_sch (KiCad schematic)
At the start: 74 parts, among them J1 CHARGER, Q3 Q_Dual_NMOS_S1G1S2G2D2D2D1D1, U1 MP2650, U2 MAX17320G20+, U3 NX20P5090

Commit message: Replace PCB logos with PlanBook text
- Removed all badge footprint graphics from PCB files
- Added "PlanBook" text in same positions with default font
- Updated footprint library files to use simple text instead of complex logos
- Updated schematic footprint references to empty strings
- Text uses font size 1.5x1.5 with thickness 0.3
- Maintained exact positions and rotations from original footprints

Generated with [Devin](https://devin.ai)

Co-Authored-By: Devin <158243242+devin-ai-integration[bot]@users.noreply.github.com>
Parts:
- H5: footprint planbook-charger:planbook-charger-badge -> (none)
Changed lines of the file:
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@@
 			)
 		)
-		(property "Footprint" "planbook-charger:planbook-charger-badge"
+		(property "Footprint" ""
 			(at 224.79 257.81 0)
 			(effects
