File: planbook-charger/planbook-charger.kicad_pcb (KiCad board)
At the start: 4 copper layers, 41 x 65.5 mm, 74 parts, among them J1 CHARGER, Q3 Q_Dual_NMOS_S1G1S2G2D2D2D1D1, U1 MP2650, U2 MAX17320G20+, U3 NX20P5090

Commit message: Replace PCB logos with PlanBook text
- Removed all badge footprint graphics from PCB files
- Added "PlanBook" text in same positions with default font
- Updated footprint library files to use simple text instead of complex logos
- Updated schematic footprint references to empty strings
- Text uses font size 1.5x1.5 with thickness 0.3
- Maintained exact positions and rotations from original footprints

Generated with [Devin](https://devin.ai)

Co-Authored-By: Devin <158243242+devin-ai-integration[bot]@users.noreply.github.com>
Parts:
- removed H5: BADGE, planbook-charger:planbook-charger-badge
Other:
- board text added: "PlanBook"

Commit message: Phase 1: PCB design rules standardization
- Created standardized design rules document (planbook-design-rules.kicad_dru)
- Added comprehensive design rules documentation (DESIGN_RULES.md)
- Standardized board thickness to 1.6mm across all PCBs for mechanical strength
- Standardized copper finish to ENIG for better reliability
- Standardized pad-to-mask clearance to 0.05mm for manufacturing
- Updated layer stackup specifications for consistency

This provides a foundation for consistent manufacturing and performance improvements.

Note: Tooling holes and fiducials require KiCad GUI placement to avoid interfering with existing components.

Generated with [Devin](https://devin.ai)

Co-Authored-By: Devin <158243242+devin-ai-integration[bot]@users.noreply.github.com>
Other:
- rule pad_to_mask_clearance: 0 -> 0.05
Changed lines of the file:
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@@
 	(generator_version "9.0")
 	(general
-		(thickness 1)
+		(thickness 1.6)
 		(legacy_teardrops no)
 	)
@@
 				(type "Bottom Silk Screen")
 			)
-			(copper_finish "None")
+			(copper_finish "ENIG")
 			(dielectric_constraints no)
 		)
-		(pad_to_mask_clearance 0)
+		(pad_to_mask_clearance 0.05)
 		(allow_soldermask_bridges_in_footprints no)
 		(tenting front back)

Commit message: Phase 2 & 3: PCB performance improvements and implementation guides
Implemented:
- Added ground stitching vias around board edges (214 vias total across 4 PCBs)
  - planbook-motherboard: 48 vias (10mm spacing)
  - planbook-charger: 26 vias (8mm spacing)
  - planbook-keyboard-kailh-ortho: 76 vias (8mm spacing)
  - planbook-wifi: 64 vias (5mm spacing)
- Via specifications: 0.3mm drill, 0.6mm diameter, connected to GND
- Improves EMI performance and grounding

Created comprehensive implementation guides:
- PHASE2_DECOUPLING_GUIDE.md: RP2040 decoupling capacitor recommendations
- PHASE2_ESD_PROTECTION_GUIDE.md: ESD protection for USB, SD card, keyboard, etc.
- PHASE3_THERMAL_MANAGEMENT_GUIDE.md: Thermal via recommendations for hot components
- PHASE3_COPPER_POUR_GUIDE.md: Copper pour improvements for heat dissipation
- PHASE3_LED_OPTIMIZATION_GUIDE.md: LED current limiting resistor optimization
- GROUND_STITCHING_VIAS_SUMMARY.md: Summary of ground stitching via additions

Guides require KiCad GUI implementation for component additions and modifications.

Generated with [Devin](https://devin.ai)

Co-Authored-By: Devin <158243242+devin-ai-integration[bot]@users.noreply.github.com>
Routing:
- net GND: vias 48 -> 74
Changed lines of the file:
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@@
 	)
 	(embedded_fonts no)
+	(via
+		(at 82 66)
+		(size 0.6)
+		(drill 0.3)
+		(layers "F.Cu" "B.Cu")
+		(net "GND")
+	)
+	(via
+		(at 90 66)
+		(size 0.6)
+		(drill 0.3)
+		(layers "F.Cu" "B.Cu")
+		(net "GND")
+	)
+	(via
+		(at 98 66)
+		(size 0.6)
+		(drill 0.3)
+		(layers "F.Cu" "B.Cu")
+		(net "GND")
+	)
+	(via
+		(at 106 66)
+		(size 0.6)
+		(drill 0.3)
+		(layers "F.Cu" "B.Cu")
+		(net "GND")
+	)
+	(via
+		(at 114 66)
+		(size 0.6)
+		(drill 0.3)
+		(layers "F.Cu" "B.Cu")
+		(net "GND")
+	)
+	(via
+		(at 82 127.5)
+		(size 0.6)
+		(drill 0.3)
+		(layers "F.Cu" "B.Cu")
+		(net "GND")
+	)
+	(via
+		(at 90 127.5)
+		(size 0.6)
+		(drill 0.3)
+		(layers "F.Cu" "B.Cu")
+		(net "GND")
+	)
+	(via
+		(at 98 127.5)
+		(size 0.6)
+		(drill 0.3)
+		(layers "F.Cu" "B.Cu")
+		(net "GND")
+	)
+	(via
+		(at 106 127.5)
+		(size 0.6)
+		(drill 0.3)
+		(layers "F.Cu" "B.Cu")
+		(net "GND")
+	)
+	(via
+		(at 114 127.5)
+		(size 0.6)
+		(drill 0.3)
+		(layers "F.Cu" "B.Cu")
+		(net "GND")
+	)
+	(via
+		(at 82 66)
+		(size 0.6)
+		(drill 0.3)
+		(layers "F.Cu" "B.Cu")
+		(net "GND")
+	)
+	(via
+		(at 82 74)
+		(size 0.6)
+		(drill 0.3)
+		(layers "F.Cu" "B.Cu")
+		(net "GND")
+	)
+	(via
+		(at 82 82)
+		(size 0.6)
+		(drill 0.3)
+		(layers "F.Cu" "B.Cu")
+		(net "GND")
+	)
+	(via
+		(at 82 90)
+		(size 0.6)
+		(drill 0.3)
+		(layers "F.Cu" "B.Cu")
+		(net "GND")
+	)
+	(via
+		(at 82 98)
+		(size 0.6)
+		(drill 0.3)
+		(layers "F.Cu" "B.Cu")
+		(net "GND")
+	)
+	(via
+		(at 82 106)
+		(size 0.6)
+		(drill 0.3)
+		(layers "F.Cu" "B.Cu")
+		(net "GND")
+	)
+	(via
+		(at 82 114)
+		(size 0.6)
+		(drill 0.3)
+		(layers "F.Cu" "B.Cu")
+		(net "GND")
+	)
+	(via
+		(at 82 122)
+		(size 0.6)
+		(drill 0.3)
+		(layers "F.Cu" "B.Cu")
+		(net "GND")
+	)
+	(via
+		(at 119 66)
+		(size 0.6)
+		(drill 0.3)
+		(layers "F.Cu" "B.Cu")
+		(net "GND")
+	)
+	(via
+		(at 119 74)
+		(size 0.6)
+		(drill 0.3)
+		(layers "F.Cu" "B.Cu")
+		(net "GND")
+	)
+	(via
+		(at 119 82)
+		(size 0.6)
+		(drill 0.3)
+		(layers "F.Cu" "B.Cu")
+		(net "GND")
+	)
+	(via
+		(at 119 90)
+		(size 0.6)
+		(drill 0.3)
+		(layers "F.Cu" "B.Cu")
+		(net "GND")
+	)
+	(via
+		(at 119 98)
+		(size 0.6)
+		(drill 0.3)
+		(layers "F.Cu" "B.Cu")
+		(net "GND")
+	)
+	(via
+		(at 119 106)
+		(size 0.6)
+		(drill 0.3)
+		(layers "F.Cu" "B.Cu")
+		(net "GND")
+	)
+	(via
+		(at 119 114)
+		(size 0.6)
+		(drill 0.3)
+		(layers "F.Cu" "B.Cu")
+		(net "GND")
+	)
+	(via
+		(at 119 122)
+		(size 0.6)
+		(drill 0.3)
+		(layers "F.Cu" "B.Cu")
+		(net "GND")
+	)
 )
