File: planbook-headphones/planbook-headphones.kicad_sch (KiCad schematic)
At the start: 15 parts, among them J1 CONN_HEAD, J2 SJ-43516-SMT, J4 CONN_PWRSW, SW1 SW_DIP_x01

Commit message: Replace PCB logos with PlanBook text
- Removed all badge footprint graphics from PCB files
- Added "PlanBook" text in same positions with default font
- Updated footprint library files to use simple text instead of complex logos
- Updated schematic footprint references to empty strings
- Text uses font size 1.5x1.5 with thickness 0.3
- Maintained exact positions and rotations from original footprints

Generated with [Devin](https://devin.ai)

Co-Authored-By: Devin <158243242+devin-ai-integration[bot]@users.noreply.github.com>
Parts:
- GFX1: footprint footprints:pref-headset-badge -> (none)
Changed lines of the file:
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@@
       (effects (font (size 1.27 1.27)) (justify left))
     )
-    (property "Footprint" "footprints:pref-headset-badge" (at 67.31 100.33 0)
+    (property "Footprint" "" (at 67.31 100.33 0)
       (effects (font (size 1.27 1.27)) hide)
     )
