File: planbook-headphones/planbook-headphones.kicad_pcb (KiCad board)
At the start: 2 copper layers, 17.6 x 95 mm, 15 parts, among them J1 CONN_HEAD, J2 SJ-43516-SMT, J4 CONN_PWRSW, SW1 SW_DIP_x01

Commit message: Replace PCB logos with PlanBook text
- Removed all badge footprint graphics from PCB files
- Added "PlanBook" text in same positions with default font
- Updated footprint library files to use simple text instead of complex logos
- Updated schematic footprint references to empty strings
- Text uses font size 1.5x1.5 with thickness 0.3
- Maintained exact positions and rotations from original footprints

Generated with [Devin](https://devin.ai)

Co-Authored-By: Devin <158243242+devin-ai-integration[bot]@users.noreply.github.com>
Parts:
- removed GFX1: BADGE, footprints:pref-headset-badge
Other:
- board text added: "PlanBook"

Commit message: Phase 1: PCB design rules standardization
- Created standardized design rules document (planbook-design-rules.kicad_dru)
- Added comprehensive design rules documentation (DESIGN_RULES.md)
- Standardized board thickness to 1.6mm across all PCBs for mechanical strength
- Standardized copper finish to ENIG for better reliability
- Standardized pad-to-mask clearance to 0.05mm for manufacturing
- Updated layer stackup specifications for consistency

This provides a foundation for consistent manufacturing and performance improvements.

Note: Tooling holes and fiducials require KiCad GUI placement to avoid interfering with existing components.

Generated with [Devin](https://devin.ai)

Co-Authored-By: Devin <158243242+devin-ai-integration[bot]@users.noreply.github.com>
Other:
- rule pad_to_mask_clearance: 0 -> 0.05
Changed lines of the file:
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@@
 (kicad_pcb (version 20221018) (generator pcbnew)
   (general
-    (thickness 1)
+    (thickness 1.6)
   )
   (paper "A4")
@@
       (layer "B.Paste" (type "Bottom Solder Paste"))
       (layer "B.SilkS" (type "Bottom Silk Screen"))
-      (copper_finish "None")
+      (copper_finish "ENIG")
       (dielectric_constraints no)
     )
-    (pad_to_mask_clearance 0)
+    (pad_to_mask_clearance 0.05)
     (pcbplotparams
       (layerselection 0x00010fc_ffffffff)
