File: planbook-motherboard/planbook-motherboard.kicad_pcb (KiCad board)
At the start: 6 copper layers, 151 x 88 mm, 441 parts, among them J1 CHARGER, J10 1-2199230-6, J11 Conn_01x33, J12 2199230-5, J13 3-2328724-1, J14 USB_C_Receptacle, J15 CONN_SPK, J16 SAMTEC_TSM-106-02-X-SH-A, J17 POWSW, J18 CONN_HEAD, J2 DM3AT-SF-PEJM5, J20 QWIIC, J3 USB_C_Receptacle, J4 09452812561, J5 SYSCTL, J6 USB_INT1, J7 HDMI_D_1.4, J8 SIM_Card, J9 Conn_01x20, SW1 SW_DIP_x01, SW2 RESET, SW3 RESET, U1 reform2-som-connector, U10 W25Q32JVSS, U11 PCF8523T, U12 AP22615AWU-7, U13 TXS0108EPW, U14 SN74AVC1T45, U15 TPD4E02B04DQA, U16 TPD4E02B04DQA, U17 TPD12S521, U18 TLV320AIC3100, U19 TPD4E02B04DQA, U2 TS3USB30EDGSR, U20 TPD4E02B04DQA, U21 TPD4E02B04DQA, U22 TPD4E02B04DQA, U23 FUSB302BMPX, U24 TXS0108EPW, U25 TUSB8041, U27 TVS2200DRV, U28 LM62460, U29 AP22615AWU-7, U3 LM2830XQMFE/NOPB, U30 TS3USB30EDGSR, U31 TS3USB30EDGSR, U32 AP22615AWU-7, U33 AT24CS02-STUM, U34 PCA9536DP, U35 TMUXHS4446RETR, U36 AP22615AWU-7, U37 TS3USB30EDGSR, U38 CY7C65215-32LTXI, U39 PCA9557PW, U4 TLV75718PDBV, U40 AP22615AWU-7, U41 AP22615AWU-7, U42 TPS560430X3FDBVR, U5 LM73100RPWR, U6 LM62460, U7 74LVC1G34, U8 RP2040, U9 TPS7A0533PDBZ, Y1 24MHz, Y2 12MHz 12pF, Y3 32.768 kHz

Commit message: Phase 1: PCB design rules standardization
- Created standardized design rules document (planbook-design-rules.kicad_dru)
- Added comprehensive design rules documentation (DESIGN_RULES.md)
- Standardized board thickness to 1.6mm across all PCBs for mechanical strength
- Standardized copper finish to ENIG for better reliability
- Standardized pad-to-mask clearance to 0.05mm for manufacturing
- Updated layer stackup specifications for consistency

This provides a foundation for consistent manufacturing and performance improvements.

Note: Tooling holes and fiducials require KiCad GUI placement to avoid interfering with existing components.

Generated with [Devin](https://devin.ai)

Co-Authored-By: Devin <158243242+devin-ai-integration[bot]@users.noreply.github.com>
Other:
- rule pad_to_mask_clearance: 0 -> 0.05
Changed lines of the file:
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@@
 	(generator_version "10.0")
 	(general
-		(thickness 1)
+		(thickness 1.6)
 		(legacy_teardrops no)
 	)
@@
 				(color "White")
 			)
-			(copper_finish "Immersion silver")
+			(copper_finish "ENIG")
 			(dielectric_constraints no)
 		)
-		(pad_to_mask_clearance 0)
+		(pad_to_mask_clearance 0.05)
 		(allow_soldermask_bridges_in_footprints no)
 		(tenting
