File: planbook-wifi/nref-wifi-m2.kicad_pcb (KiCad board)
At the start: 4 copper layers, 66 x 24 mm, 36 parts, among them J1 Bus_M.2_Socket_E, J2 Conn_01x20, U1 TPS62A04ABDRL, X1 ECS-327MVATX-2-CN-TR3

Commit message: Replace PCB logos with PlanBook text
- Removed all badge footprint graphics from PCB files
- Added "PlanBook" text in same positions with default font
- Updated footprint library files to use simple text instead of complex logos
- Updated schematic footprint references to empty strings
- Text uses font size 1.5x1.5 with thickness 0.3
- Maintained exact positions and rotations from original footprints

Generated with [Devin](https://devin.ai)

Co-Authored-By: Devin <158243242+devin-ai-integration[bot]@users.noreply.github.com>
Parts:
- removed H4: LOGO, footprints:nref-wifi-m2-badge
Other:
- board text added: "PlanBook"
