File: planbook-wifi/planbook-wifi.kicad_sch (KiCad schematic)
At the start: 9 parts, among them J21 CONN_HEAD, J22 SJ-43516-SMT, J24 CONN_PWRSW, SW21 SW_DIP_x01

Commit message: Replace PCB logos with PlanBook text
- Removed all badge footprint graphics from PCB files
- Added "PlanBook" text in same positions with default font
- Updated footprint library files to use simple text instead of complex logos
- Updated schematic footprint references to empty strings
- Text uses font size 1.5x1.5 with thickness 0.3
- Maintained exact positions and rotations from original footprints

Generated with [Devin](https://devin.ai)

Co-Authored-By: Devin <158243242+devin-ai-integration[bot]@users.noreply.github.com>
Parts:
- GFX21: footprint footprints:pref-headset-badge -> (none)
Changed lines of the file:
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@@
 			)
 		)
-		(property "Footprint" "footprints:pref-headset-badge"
+		(property "Footprint" ""
 			(at 67.31 100.33 0)
 			(effects
