File: planbook-wifi/planbook-wifi.kicad_pcb (KiCad board)
At the start: 4 copper layers, 27.6 x 95 mm, 42 parts, among them J1 Bus_M.2_Socket_E, J2 Conn_01x20, J21 CONN_HEAD, J22 SJ-43516-SMT, J24 CONN_PWRSW, SW21 SW_DIP_x01, U1 TPS62A04ABDRL, X1 ECS-327MVATX-2-CN-TR3

Commit message: Replace PCB logos with PlanBook text
- Removed all badge footprint graphics from PCB files
- Added "PlanBook" text in same positions with default font
- Updated footprint library files to use simple text instead of complex logos
- Updated schematic footprint references to empty strings
- Text uses font size 1.5x1.5 with thickness 0.3
- Maintained exact positions and rotations from original footprints

Generated with [Devin](https://devin.ai)

Co-Authored-By: Devin <158243242+devin-ai-integration[bot]@users.noreply.github.com>
Parts:
- removed GFX21: BADGE, footprints:pref-headset-badge-r3
Other:
- board text added: "PlanBook"

Commit message: Phase 1: PCB design rules standardization
- Created standardized design rules document (planbook-design-rules.kicad_dru)
- Added comprehensive design rules documentation (DESIGN_RULES.md)
- Standardized board thickness to 1.6mm across all PCBs for mechanical strength
- Standardized copper finish to ENIG for better reliability
- Standardized pad-to-mask clearance to 0.05mm for manufacturing
- Updated layer stackup specifications for consistency

This provides a foundation for consistent manufacturing and performance improvements.

Note: Tooling holes and fiducials require KiCad GUI placement to avoid interfering with existing components.

Generated with [Devin](https://devin.ai)

Co-Authored-By: Devin <158243242+devin-ai-integration[bot]@users.noreply.github.com>
Other:
- rule pad_to_mask_clearance: 0 -> 0.05
Changed lines of the file:
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@@
 	(generator_version "10.0")
 	(general
-		(thickness 1)
+		(thickness 1.6)
 		(legacy_teardrops no)
 	)
@@
 				(type "Bottom Silk Screen")
 			)
-			(copper_finish "None")
+			(copper_finish "ENIG")
 			(dielectric_constraints no)
 		)
-		(pad_to_mask_clearance 0)
+		(pad_to_mask_clearance 0.05)
 		(allow_soldermask_bridges_in_footprints no)
 		(tenting

Commit message: Phase 2 & 3: PCB performance improvements and implementation guides
Implemented:
- Added ground stitching vias around board edges (214 vias total across 4 PCBs)
  - planbook-motherboard: 48 vias (10mm spacing)
  - planbook-charger: 26 vias (8mm spacing)
  - planbook-keyboard-kailh-ortho: 76 vias (8mm spacing)
  - planbook-wifi: 64 vias (5mm spacing)
- Via specifications: 0.3mm drill, 0.6mm diameter, connected to GND
- Improves EMI performance and grounding

Created comprehensive implementation guides:
- PHASE2_DECOUPLING_GUIDE.md: RP2040 decoupling capacitor recommendations
- PHASE2_ESD_PROTECTION_GUIDE.md: ESD protection for USB, SD card, keyboard, etc.
- PHASE3_THERMAL_MANAGEMENT_GUIDE.md: Thermal via recommendations for hot components
- PHASE3_COPPER_POUR_GUIDE.md: Copper pour improvements for heat dissipation
- PHASE3_LED_OPTIMIZATION_GUIDE.md: LED current limiting resistor optimization
- GROUND_STITCHING_VIAS_SUMMARY.md: Summary of ground stitching via additions

Guides require KiCad GUI implementation for component additions and modifications.

Generated with [Devin](https://devin.ai)

Co-Authored-By: Devin <158243242+devin-ai-integration[bot]@users.noreply.github.com>
Routing:
- net GND: vias 76 -> 140
